File: 87keyboard.kicad_sch (KiCad schematic)
At the start: 420 parts, among them J1 USB_C_Receptacle_USB2.0, J2 Conn_01x04, J3 Conn_01x08, J4 Conn_01x04, J5 SM04B-SRSS-TB(LF)(SN), J6 SM04B-SRSS-TB(LF)(SN), J7 Conn_01x03, J8 Conn_01x04, J9 SM04B-SRSS-TB(LF)(SN), Q1 DTC123JKAT146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

Commit message: prepare rev 1.1
Parts:
- removed C106: 100n, Capacitor_SMD:C_0402_1005Metric, symbol Device:C_Small
- C7: Specification (none) -> 25V 10% X7R 0402
Other:
- moved on the sheet: C107, D176, J5, J6, J9, Q1, R10, R11, R12, R13, R9, SW1
